File: PCB/Macropad v2.kicad_pcb (KiCad board)
At the start: 2 copper layers, 87.5 x 84 mm, 27 parts, among them J1 Conn_01x04_Pin, SW1 SW_Push, SW10 SW_Push, SW11 SW_Push, SW12 SW_Push, SW2 SW_Push, SW3 SW_Push, SW4 SW_Push, SW5 SW_Push, SW6 SW_Push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

Commit message: Final files of Keybie
Updated CASE, PCB and firmware
Routing:
- net Row1: track 99.5 -> 78.6 mm
- net Net-(D6-PadA): track 27.5 -> 13.4 mm
- net Net-(D9-PadA): track 14.8 -> 13.3 mm
Other:
- board text added: "Pranavi's Macropad :) Keybie!"
- board text added: "↓"
- board text removed: "Pranavi Alla's Macropad :)"
